File: hardware/RevA/RevA.kicad_pcb (KiCad board)
At the start: 4 copper layers, 85 x 54 mm, 145 parts, among them J1 USB_C_Receptacle_USB2.0, J2 DNP Conn_02x02_Odd_Even, J3 DNP Conn_01x02, J4 DNP Conn_02x03_Odd_Even, J5 DNP Conn_01x02, SW1 SW_Push, SW2 SW_Push, U1 SY8120B1ABC, U10 SPI RAM LY68L6400SLIT, U2 XC6206P25, U3 SY8120B1ABC, U4 SPI Flash W25Q128JVSIQ, U5 MIMXRT1011DAE5A, U6 MAX803SQ308T1G, U7 SPI RAM LY68L6400SLIT, U8 LFE5U-12F-6BG256C, U9 16MHz 20ppm, Y1 24MHz 10ppm

Commit message: Dual source design from Digikey/Mouser, rev 0.2R
Adjustable Reg -> AP3211KTR-G1 + Freewheel Diode
Fixed Reg -> AP2120N-2.5TRG1
24MHz Crystal -> Epson TSX-3225
16MHz OSC -> ECS-3225MV
USB Connector -> CUI UJ31-CH-31-SMT-TR
RGB LED -> Cree CLMVC-FKA
Parts:
- added D10: Schottky, Diode_SMD:D_SOD-323F, F.Cu at (123.2, 51.8)
- added D11: Schottky, Diode_SMD:D_SOD-323F, F.Cu at (104.7, 59.4)
- added R38: 1kΩ, Resistor_SMD:R_0402_1005Metric, B.Cu at (132.7, 81.1)
- C1, C20, C23, C3, C30, C31, C32, C33, C34, C35, C36, C37, C38, C39, C40, C41, C42, C43, C44: value 100n -> 100nF
- C10, C15, C4: value 4u7 -> 4.7µF
- C11, C14: value 20p -> 18pF
- C12, C25, C26, C27, C28, C29, C6, C7: value 22u -> 22µF
- C13, C18, C19, C2, C5, C8, C9: value 220n -> 220nF
- C16, C17: value 100n -> 10nF
- C21, C22: value 22p -> 18pF
- C24: value 10u -> 10µF
- D1: value LED_ARGB -> CLMVC-FKA-CL1D1L71BB7C3C3
- J1: value USB_C_Receptacle_USB2.0 -> UJ31-CH-31-SMT-TR; footprint Connector_USB_Extra:USB_C_Receptacle_GT-USB-7010 -> ecp5board:CUI_UJ31-CH-312-SMT-TR
- L1, L2, L3: value 4u7 1A -> 4.7µH 1A
- R1: value 100K -> 0Ω
- R10: value 18K -> 33kΩ
- R11, R9: value 15K -> 15kΩ
- R12: value 3K3 -> 4.7kΩ
- R13, R14, R15, R16, R17, R2, R25, R26, R27, R28, R29, R3, R30, R31, R32: value 10K -> 10kΩ
- R18, R19, R23, R24, R33, R34, R5: value 4K7 -> 4.7kΩ
- R20: value 10K -> 4.7kΩ
- R21, R22: value 10K -> 1kΩ
- R36, R37, R4: value 1K -> 1kΩ
- R6, R7: value 5K1 -> 5.1kΩ
- R8: value 30K -> 33kΩ
- RN1, RN10, RN2, RN3, RN4, RN5, RN6, RN7, RN8, RN9: footprint Resistor_SMD:R_Array_Convex_4x0603 -> Resistor_SMD:R_Array_Convex_4x0402
- U1, U3: value SY8120B1ABC -> AP3211KTR-G1
- U10, U7: value SPI RAM LY68L6400SLIT -> SERIAL SRAM, 4MB
- U2: value XC6206P25 -> AP2120N-2.5
- U9: value 16MHz 20ppm -> 16MHz ±25ppm
- moved J1 4.58 mm to (109.2, 76.5)
- moved C17 3.04 mm to (106.8, 57.8)
- moved R22 2.25 mm to (105.0, 92.8)
- moved R20 2.20 mm to (105.0, 95.0)
- moved C16 2.13 mm to (121.0, 51.8), turned to 90 degrees
- moved R1 1.35 mm to (101.5, 69.5), turned to -90 degrees
- moved C18 0.66 mm to (114.2, 71.7)
- moved C20 0.61 mm to (113.3, 75.2)
- moved C24 0.59 mm to (113.3, 74.2)
- moved C11 0.56 mm to (113.3, 79.8)
- moved C13 0.56 mm to (113.3, 78.8)
- moved C15 0.56 mm to (113.3, 77.8)
- moved FB1 0.50 mm to (107.2, 70.2)
- moved R6 0.15 mm to (104.5, 70.2)
- moved R7 0.15 mm to (103.5, 70.2)
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Connections:
- net Net-(C19-Pad2) renamed /DCDC_PSWITCH
- J1 pad A8: (no net) -> Net-(J1-PadA8)
- J1 pad B8: (no net) -> Net-(J1-PadB8)
- R1 pad 1: /USB_SHIELD -> GND
- R1 pad 2: GND -> /USB_SHIELD
- R20 pad 2: Net-(D1-Pad2) -> Net-(D1-Pad4)
- R22 pad 2: Net-(D1-Pad4) -> Net-(D1-Pad2)
- U5 pad 1: (no net) -> Net-(U5-Pad1)
- U5 pad 21: (no net) -> Net-(U5-Pad21)
- U5 pad 24: (no net) -> Net-(U5-Pad24)
- U5 pad 28: (no net) -> Net-(U5-Pad28)
- U5 pad 36: (no net) -> Net-(U5-Pad36)
- U5 pad 4: (no net) -> Net-(U5-Pad4)
- U5 pad 43: (no net) -> Net-(U5-Pad43)
- U5 pad 46: (no net) -> Net-(U5-Pad46)
- U5 pad 47: (no net) -> Net-(U5-Pad47)
- U5 pad 48: (no net) -> Net-(U5-Pad48)
- U5 pad 49: (no net) -> Net-(U5-Pad49)
- U5 pad 5: (no net) -> Net-(U5-Pad5)
- U5 pad 6: (no net) -> Net-(U5-Pad6)
- U5 pad 79: (no net) -> Net-(U5-Pad79)
- U5 pad 8: (no net) -> Net-(U5-Pad8)
- U5 pad 80: (no net) -> Net-(U5-Pad80)
- U5 pad 9: (no net) -> Net-(U5-Pad9)
- U8 pad A6: (no net) -> Net-(U8-PadA6)
- U8 pad B5: (no net) -> Net-(U8-PadB5)
- U8 pad C10: (no net) -> Net-(U8-PadC10)
- U8 pad C11: (no net) -> Net-(U8-PadC11)
- U8 pad C12: (no net) -> Net-(U8-PadC12)
- U8 pad C13: (no net) -> Net-(U8-PadC13)
- U8 pad C14: (no net) -> Net-(U8-PadC14)
- U8 pad C3: (no net) -> Net-(U8-PadC3)
- U8 pad C5: (no net) -> Net-(U8-PadC5)
- U8 pad C8: (no net) -> Net-(U8-PadC8)
- U8 pad C9: (no net) -> Net-(U8-PadC9)
- U8 pad D10: (no net) -> Net-(U8-PadD10)
- U8 pad D11: (no net) -> Net-(U8-PadD11)
- U8 pad D12: (no net) -> Net-(U8-PadD12)
- U8 pad D13: (no net) -> Net-(U8-PadD13)
- U8 pad D14: (no net) -> Net-(U8-PadD14)
- U8 pad D3: (no net) -> Net-(U8-PadD3)
- U8 pad D5: (no net) -> Net-(U8-PadD5)
- U8 pad D6: (no net) -> Net-(U8-PadD6)
- U8 pad D7: (no net) -> Net-(U8-PadD7)
- U8 pad D8: (no net) -> Net-(U8-PadD8)
- U8 pad D9: (no net) -> Net-(U8-PadD9)
- U8 pad E1: (no net) -> Net-(U8-PadE1)
- U8 pad E10: (no net) -> Net-(U8-PadE10)
- U8 pad E11: (no net) -> Net-(U8-PadE11)
- U8 pad E12: (no net) -> Net-(U8-PadE12)
- U8 pad E13: (no net) -> Net-(U8-PadE13)
- U8 pad E14: (no net) -> Net-(U8-PadE14)
- U8 pad E3: (no net) -> Net-(U8-PadE3)
- U8 pad E4: (no net) -> Net-(U8-PadE4)
- U8 pad E5: (no net) -> Net-(U8-PadE5)
- U8 pad E6: (no net) -> Net-(U8-PadE6)
- U8 pad E7: (no net) -> Net-(U8-PadE7)
- U8 pad E8: (no net) -> Net-(U8-PadE8)
- U8 pad E9: (no net) -> Net-(U8-PadE9)
- U8 pad F12: (no net) -> Net-(U8-PadF12)
- U8 pad F13: (no net) -> Net-(U8-PadF13)
- U8 pad F2: (no net) -> Net-(U8-PadF2)
- U8 pad F3: (no net) -> Net-(U8-PadF3)
- U8 pad F4: (no net) -> Net-(U8-PadF4)
- U8 pad F5: (no net) -> Net-(U8-PadF5)
- U8 pad G12: (no net) -> Net-(U8-PadG12)
- U8 pad G13: (no net) -> Net-(U8-PadG13)
- U8 pad G14: (no net) -> Net-(U8-PadG14)
- U8 pad G3: (no net) -> Net-(U8-PadG3)
- U8 pad G4: (no net) -> Net-(U8-PadG4)
- U8 pad G5: (no net) -> Net-(U8-PadG5)
- U8 pad H12: (no net) -> Net-(U8-PadH12)
- U8 pad H13: (no net) -> Net-(U8-PadH13)
- U8 pad H14: (no net) -> Net-(U8-PadH14)
- U8 pad H3: (no net) -> Net-(U8-PadH3)
- U8 pad H4: (no net) -> Net-(U8-PadH4)
- U8 pad H5: (no net) -> Net-(U8-PadH5)
- U8 pad J12: (no net) -> Net-(U8-PadJ12)
- U8 pad J13: (no net) -> Net-(U8-PadJ13)
- U8 pad J14: (no net) -> Net-(U8-PadJ14)
- U8 pad J3: (no net) -> Net-(U8-PadJ3)
- U8 pad J4: (no net) -> Net-(U8-PadJ4)
- U8 pad J5: (no net) -> Net-(U8-PadJ5)
- U8 pad K1: (no net) -> Net-(U8-PadK1)
- U8 pad K12: (no net) -> Net-(U8-PadK12)
- U8 pad K13: (no net) -> Net-(U8-PadK13)
- U8 pad K14: (no net) -> Net-(U8-PadK14)
- U8 pad K15: (no net) -> Net-(U8-PadK15)
- U8 pad K16: (no net) -> Net-(U8-PadK16)
- U8 pad K2: (no net) -> Net-(U8-PadK2)
- U8 pad K3: (no net) -> Net-(U8-PadK3)
- U8 pad K4: (no net) -> Net-(U8-PadK4)
- U8 pad K5: (no net) -> Net-(U8-PadK5)
- U8 pad L12: (no net) -> Net-(U8-PadL12)
- U8 pad L13: (no net) -> Net-(U8-PadL13)
- U8 pad L14: (no net) -> Net-(U8-PadL14)
- U8 pad L3: (no net) -> Net-(U8-PadL3)
- U8 pad L4: (no net) -> Net-(U8-PadL4)
- U8 pad L5: (no net) -> Net-(U8-PadL5)
- U8 pad M11: (no net) -> Net-(U8-PadM11)
- U8 pad M12: (no net) -> Net-(U8-PadM12)
- U8 pad M13: (no net) -> Net-(U8-PadM13)
- U8 pad M15: (no net) -> Net-(U8-PadM15)
- U8 pad M16: (no net) -> Net-(U8-PadM16)
- U8 pad M2: (no net) -> Net-(U8-PadM2)
- U8 pad M3: (no net) -> Net-(U8-PadM3)
- U8 pad M4: (no net) -> Net-(U8-PadM4)
- U8 pad M5: (no net) -> Net-(U8-PadM5)
- U8 pad M6: (no net) -> Net-(U8-PadM6)
- U8 pad M8: (no net) -> Net-(U8-PadM8)
- U8 pad M9: (no net) -> Net-(U8-PadM9)
- U8 pad N11: (no net) -> Net-(U8-PadN11)
- U8 pad N12: (no net) -> Net-(U8-PadN12)
- U8 pad N13: (no net) -> Net-(U8-PadN13)
- U8 pad N14: (no net) -> Net-(U8-PadN14)
- U8 pad N16: (no net) -> Net-(U8-PadN16)
- U8 pad N3: (no net) -> Net-(U8-PadN3)
- U8 pad N4: (no net) -> Net-(U8-PadN4)
- U8 pad N5: (no net) -> Net-(U8-PadN5)
- U8 pad N6: (no net) -> Net-(U8-PadN6)
- U8 pad P12: (no net) -> Net-(U8-PadP12)
- U8 pad P13: (no net) -> Net-(U8-PadP13)
- U8 pad P14: (no net) -> Net-(U8-PadP14)
- U8 pad P15: (no net) -> Net-(U8-PadP15)
- U8 pad P3: (no net) -> Net-(U8-PadP3)
- U8 pad P4: (no net) -> Net-(U8-PadP4)
- U8 pad P5: (no net) -> Net-(U8-PadP5)
- U8 pad P6: (no net) -> Net-(U8-PadP6)
- U8 pad P7: (no net) -> Net-(U8-PadP7)
- U8 pad P8: (no net) -> Net-(U8-PadP8)
- U8 pad R12: (no net) -> Net-(U8-PadR12)
- U8 pad R13: (no net) -> Net-(U8-PadR13)
- U8 pad R14: (no net) -> Net-(U8-PadR14)
- U8 pad R15: (no net) -> Net-(U8-PadR15)
- U8 pad R16: (no net) -> Net-(U8-PadR16)
- U8 pad R5: (no net) -> Net-(U8-PadR5)
- U8 pad R6: (no net) -> Net-(U8-PadR6)
- U8 pad R7: (no net) -> Net-(U8-PadR7)
- U8 pad T13: (no net) -> Net-(U8-PadT13)
- U8 pad T14: (no net) -> Net-(U8-PadT14)
- U8 pad T15: (no net) -> Net-(U8-PadT15)
- U8 pad T6: (no net) -> Net-(U8-PadT6)
Routing:
- net Net-(C17-Pad1): track 1.60 -> 5.15 mm
- net GND: track 151.4 -> 154.9 mm, vias 94 -> 93
- net Net-(J1-PadA5): track 7.78 -> 10.6 mm, vias 0 -> 2
- net /VBUS_UNFILTERED: track 5.44 -> 7.87 mm
- net Net-(J1-PadB5): track 10.3 -> 8.11 mm
- net Net-(C16-Pad2): track 1.67 -> 3.69 mm
- net /USB_DM: track 12.2 -> 10.4 mm, vias 0 -> 1
- net /PMOD2_1: track 2.69 -> 4.12 mm
- net /PMOD3_1: track 2.66 -> 3.95 mm
- net /PMOD4_3: track 2.69 -> 3.95 mm
- net /PMOD3_3: track 2.64 -> 3.90 mm
- net /FPGA_~HOLD: track 21.3 -> 22.5 mm
- net /PMOD3_4: track 2.64 -> 3.80 mm
- net /PMOD4_4: track 2.68 -> 3.79 mm
- net /LED_R: track 35.0 -> 36.1 mm
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Other:
- rule pad_to_mask_clearance: 0.051 -> 0
- board text added: "2R"
