File: hardware/RevA/RevA.kicad_sch (KiCad schematic)
At the start: 145 parts, among them J1 USB_C_Receptacle_USB2.0, J2 DNP Conn_02x02_Odd_Even, J3 DNP Conn_01x02, J4 DNP Conn_02x03_Odd_Even, J5 DNP Conn_01x02, SW1 SW_Push, SW2 SW_Push, U1 SY8120B1ABC, U10 SPI RAM LY68L6400SLIT, U2 XC6206P25, U3 SY8120B1ABC, U4 SPI Flash W25Q128JVSIQ, U5 MIMXRT1011DAE5A, U6 MAX803SQ308T1G, U7 SPI RAM LY68L6400SLIT, U8 LFE5U-12F-6BG256C, U9 16MHz 20ppm, Y1 24MHz 10ppm

Commit message: Dual source design from Digikey/Mouser, rev 0.2R
Adjustable Reg -> AP3211KTR-G1 + Freewheel Diode
Fixed Reg -> AP2120N-2.5TRG1
24MHz Crystal -> Epson TSX-3225
16MHz OSC -> ECS-3225MV
USB Connector -> CUI UJ31-CH-31-SMT-TR
RGB LED -> Cree CLMVC-FKA
Parts:
- removed D1: LED_ARGB, LED_SMD:LED_Cree-PLCC4_2x2mm_CW, symbol Device:LED_ARGB
- removed J1: USB_C_Receptacle_USB2.0, Connector_USB_Extra:USB_C_Receptacle_GT-USB-7010, symbol Connector:USB_C_Receptacle_USB2.0
- removed U1, U3: SY8120B1ABC, Package_TO_SOT_SMD:SOT-23-6, symbol SY8120B1ABC:SY8120B1ABC
- added D1: CLMVC-FKA-CL1D1L71BB7C3C3, LED_SMD:LED_Cree-PLCC4_2x2mm_CW, symbol LED_ABGR:LED_ABGR
- added D10, D11: Schottky, Diode_SMD:D_SOD-323F, symbol Device:D_Schottky_Small_ALT
- added J1: UJ31-CH-31-SMT-TR, ecp5board:CUI_UJ31-CH-312-SMT-TR, symbol Connector:USB_C_Receptacle
- added R38: 1kΩ, Resistor_SMD:R_0402_1005Metric, symbol Device:R
- added U1, U3: AP3211KTR-G1, Package_TO_SOT_SMD:SOT-23-6, symbol Regulator_Switching:AOZ1280CI
- C1, C3, C40, C43: value 100n -> 100nF
- C10, C15: value 4u7 -> 4.7µF; LCSC https://lcsc.com/product-detail/Multilayer-Ceramic-Capacito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 -> (none)
- C11, C14: value 20p -> 18pF
- C12, C25, C26, C27, C28, C29, C6, C7: value 22u -> 22µF; Digikey (none) -> 490-GRM219R61C226ME15KCT-ND; LCSC C98190 -> (none); LCSC EUR 0.0297 -> (none); LCSC URL https://lcsc.com/product-detail/Multilayer-Ceramic-Capacito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 -> (none); Mouser (none) -> 81-GRM219R61C226ME1K; PN (none) -> GRM219R61C226ME15K
- C13, C18: value 220n -> 220nF; LCSC https://lcsc.com/product-detail/Multilayer-Ceramic-Capacito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 -> (none)
- C16, C17: value 100n -> 10nF
- C19, C2, C5, C8, C9: value 220n -> 220nF
- C20, C23, C30, C31, C32, C33, C34, C35, C36, C37, C38, C39, C41, C42, C44: value 100n -> 100nF; LCSC https://lcsc.com/product-detail/Multilayer-Ceramic-Capacito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 -> (none)
- C21, C22: value 22p -> 18pF
- C24: value 10u -> 10µF; LCSC https://lcsc.com/product-detail/Multilayer-Ceramic-Capacito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 -> (none)
- C4: value 4u7 -> 4.7µF
- D2, D3, D4, D5, D6, D7, D8, D9: Digikey (none) -> 732-4978-1-ND; LCSC C84263 -> (none); LCSC EUR 0.0111 -> (none); LCSC URL https://lcsc.com/product-detail/Light-Emitting-Diodes-LED_R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 -> (none); Mouser (none) -> 710-150060RS75000; PN (none) -> 150060RS75000
- FB1: symbol Device:Ferrite_Bead -> Device:Ferrite_Bead_Small; Digikey (none) -> 490-5987-1-ND; LCSC C88993 -> (none); LCSC EUR 0.0183 -> (none); LCSC URL https://lcsc.com/product-detail/Ferrite-Beads-And-Chips_muR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 -> (none); Mouser (none) -> 81-BLM21PG220SN1D; PN (none) -> BLM21PG220SN1D
- JP1, JP2, JP3, JP4, JP5, JP6, JP7, JP8, JP9: LCSC C105871 -> (none); LCSC EUR 0.0005 -> (none); LCSC URL https://lcsc.com/product-detail/Chip-Resistor-Surface-Mount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 -> (none)
- L1, L2, L3: value 4u7 1A -> 4.7µH 1A; Digikey (none) -> 490-18407-1-ND; LCSC C90319 -> (none); LCSC EUR 0.0691 -> (none); LCSC URL https://lcsc.com/product-detail/Inductors-SMD_Taiyo-Yuden_C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 -> (none); Mouser (none) -> 81-DFE322520FD4R7MP2; PN (none) -> DFE322520FD-4R7M=P2
- PMOD1, PMOD2, PMOD3, PMOD4, PMOD5: Digikey (none) -> SAM1224-06-ND; LCSC C239357 -> (none); LCSC EUR 0.1299 -> (none); LCSC URL https://lcsc.com/product-detail/Pin-Header-Female-Header_Ch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 -> (none); Mouser (none) -> 200-SSQ10602TDRA; PN (none) -> SSQ-106-02-T-D-RA
- R1: value 100K -> 0Ω
- R10: value 18K -> 33kΩ
- R11, R9: value 15K -> 15kΩ
- R12: value 3K3 -> 4.7kΩ
- R13, R14, R15, R16, R17, R2, R25, R26, R27, R28, R29, R3, R30, R31, R32: value 10K -> 10kΩ
- R18, R19, R23, R24, R33, R34, R5: value 4K7 -> 4.7kΩ
- R20: value 10K -> 4.7kΩ
- R21, R22: value 10K -> 1kΩ
- R36, R37, R4: value 1K -> 1kΩ
- R6, R7: value 5K1 -> 5.1kΩ
- R8: value 30K -> 33kΩ
- RN1, RN10, RN2, RN3, RN4, RN5, RN6, RN7, RN8, RN9: footprint Resistor_SMD:R_Array_Convex_4x0603 -> Resistor_SMD:R_Array_Convex_4x0402; Digikey (none) -> Y7220CT-ND; LCSC C309446 -> (none); LCSC EUR 0.0075 -> (none); LCSC URL https://lcsc.com/product-detail/Others_YAGEO-AF124-JR-0722R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 -> (none); Mouser (none) -> 667-EXB-28V220JX; PN (none) -> EXB-28V220JX
- SW1, SW2: Digikey (none) -> CKN12329-1-ND; LCSC C118141 -> (none); LCSC EUR 0.0307 -> (none); LCSC URL https://lcsc.com/product-detail/Tactile-Switches_Korean-Hro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 -> (none); Mouser (none) -> 611-PTS636SM25FSMTRL; PN (none) -> PTS636 SM25F SMTR LFS
- U10, U7: value SPI RAM LY68L6400SLIT -> SERIAL SRAM, 4MB; LCSC C261881 -> (none); LCSC EUR 0.4665 -> (none); LCSC URL https://lcsc.com/product-detail/RAM_Lyontek-Inc-LY68L6400SL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 -> (none); Mouser (none) -> 870-62WS5128FBLL2NIT; PN (none) -> IS62WVS5128FBLL
- U2: value XC6206P25 -> AP2120N-2.5; Digikey (none) -> AP2120N-2.5TRG1DICT-ND; LCSC C15906 -> (none); LCSC EUR 0.0529 -> (none); LCSC URL https://lcsc.com/product-detail/Low-Dropout-Regulators-LDO_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 -> (none); Mouser (none) -> 621-AP2120N-2.5TRG1; PN (none) -> AP2120N-2.5TRG1
- U4: Digikey (none) -> W25Q128JVSIQCT-ND; LCSC C97521 -> (none); LCSC EUR 0.4692 -> (none); LCSC URL https://lcsc.com/product-detail/FLASH_Winbond-Elec-W25Q128J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 -> (none); Mouser (none) -> 454-W25Q128JVSIQTR; PN (none) -> W25Q128JVSIQ TR
- U5: Digikey (none) -> 568-MIMXRT1011DAE5A-ND; Mouser EUR 2.95 -> (none); PN (none) -> MIMXRT1011DAE5A
- U5: Digikey (none) -> 568-MIMXRT1011DAE5A-ND; Mouser URL https://www.mouser.se/ProductDetail/NXP-Semiconductors/MIMX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 -> (none); PN (none) -> MIMXRT1011DAE5A
- U6: Digikey (none) -> MAX803SQ308T1GOSCT-ND; LCSC C233650 -> (none); LCSC EUR 0.1589 -> (none); LCSC URL https://lcsc.com/product-detail/Microprocessor-Microcontrol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 -> (none); Mouser (none) -> 863-MAX803SQ308T1G; PN (none) -> MAX803SQ308T1G
- U8: Digikey (none) -> 842-LFE5U12F6BG256C; Mouser URL https://www.mouser.se/ProductDetail/Lattice/LFE5U-12F-6BG25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 -> (none); PN (none) -> LFE5U-12F-6BG256C
- U9: value 16MHz 20ppm -> 16MHz ±25ppm; Digikey (none) -> XC2883CT-ND; LCSC C387369 -> (none); LCSC EUR 0.2984 -> (none); LCSC URL https://lcsc.com/product-detail/SMD-Oscillators-XO_Shenzhen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 -> (none); Mouser (none) -> 520-3225MV-160-CNT; PN (none) -> ECS-3225MV-160-CN-TR
- Y1: Digikey (none) -> SER3634CT-ND; LCSC C164058 -> (none); LCSC EUR 0.0642 -> (none); LCSC URL https://lcsc.com/product-detail/SMD-Crystal-Resonators_Zhej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 -> (none); Mouser (none) -> 732-TX325-24F20G-AC3; PN (none) -> TSX-3225 24.0000MF20G-AC3
Connections:
- net +3V3: now also D1.1 (A)
- net FPGA_~HOLD: now also R38.2
- net GND: now also R1.1, D10.2 (A), D11.2 (A), J1.A1 (GND), J1.A12 (GND), J1.B1 (GND), J1.B12 (GND), R38.1, U1.2 (GND), U3.2 (GND); no longer R1.2
- net USB_DM: now also J1.A7 (D-), J1.B7 (D-)
- net USB_DP: now also J1.A6 (D+), J1.B6 (D+)
- net USB_SHIELD: now also R1.2, J1.S1 (SHIELD); no longer R1.1
- net VBUS: now also U1.5 (VIN), U3.5 (VIN)
- net VBUS_UNFILTERED: now also J1.A4 (VBUS), J1.A9 (VBUS), J1.B4 (VBUS), J1.B9 (VBUS)
- net at R6.1: now also J1.A5 (CC1)
- net at R7.1: now also J1.B5 (CC2)
- net at R20.2: now also D1.4 (RK)
- net at R21.2: now also D1.3 (GK)
- net at R22.2: now also D1.2 (BK)
- net at C16.2, L2.1: now also D10.1 (K), U1.6 (LX)
- net DCDC_PSWITCH: now reaches C19.2, R8.1, U5.15 (DCDC_PSWITCH)
- net at R2.2: now also U1.4 (EN)
- net at C16.1: now also U1.1 (BST)
- net at C21.1, R10.2, R9.1: now also U1.3 (FB)
- net at C17.1: now also U3.1 (BST)
- net at C22.1, R11.1, R12.2: now also U3.3 (FB)
- net at R3.2: now also U3.4 (EN)
- net at C17.2, L3.1: now also D11.1 (K), U3.6 (LX)
- no-connect marks 137 -> 145
Other:
- note added: "1V1: 1.5A max"
- note added: "2V5: 150mA max"
- note added: "3V3: 1.5A max"
- note added: "Fit 1k pull-down to allow the iMX to use the flash exclusively during boot-up"
- note added: "RevA 0.2: [X] Add strong 1K pull-ups on UART RX and TX lines. [X] Tune LED brightness. 10K looks good. [X] Add USB connector TH pads solderpaste layer. [X] Fix incorrect silkscreen for bootmode and swd. [ ] Invert and wire SW_USR to BOOT0 as well, in order to force ROM BL [ ] Replace 0R resistors on back with solderjumpers. Need to put resistors on top layer. [X] Fix incorrect RGB LED footprint, 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"
- note added: "Vout = (1 + 15/33) * 0.81 = 1.18V"
- note added: "Vout = (1 + 15/4.7) * 0.81 = 3.4V"
- note removed: "1V1: 2A max"
- note removed: "2V5: 200mA max"
- note removed: "3V3: 2A max"
- note removed: "Ra = Rb * (0.6 / (Vout - 0.6)) Vout = (1 + Ra/Rb) * 0.6"
- note removed: "RevA 0.2: [X] Add strong 1K pull-ups on UART RX and TX lines. [X] Tune LED brightness. 10K looks good. [X] Add USB connector TH pads solderpaste layer. [X] Fix incorrect silkscreen for bootmode and swd. [ ] Invert and wire SW_USR to BOOT0 as well, in order to force ROM BL [ ] Replace 0R resistors on back with solderjumpers. Need to put resistors on top layer. [ ] Fix incorrect RGB LED footprint, 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"
- note removed: "Vout = (1 + 15e3/18e3) * 0.6 = 1.1V"
- note removed: "Vout = (1 + 15e3/3.3e3) * 0.6 = 3.33V"
- company: Konrad Beckmann -> Konrad Beckmann // Modifed Richard Meadows 2020
- moved on the sheet: C1, C10, C11, C13, C14, C15, C17, C18, C2, C20, C21, C22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
